File: hardware/incur_board.kicad_pcb (KiCad board)
At the start: 2 copper layers, 100 x 100 mm, 38 parts, among them J1 mono_jack_3.5mm, J2 mono_jack_3.5mm, J3 mono_jack_3.5mm, J4 mono_jack_3.5mm, J5 din5, J6 Conn_01x01, J7 rca, J8 2x20_Extra_Tall_Header, U1 MCP3008, U2 6N138

Commit message: plot schematic
Parts:
- J1, J2, J3, J4: footprint Connections_Thonkiconn:Jack_3.5mm_QingPu_WQP-PJ398SM_Vertical_CircularHoles -> lib_fp:Jack_3.5mm_QingPu_WQP-PJ398SM_Vertical_CircularHoles
