File: hardware/i_n_c_u_r.kicad_sch (KiCad schematic)
At the start: 30 parts, among them J1 mono_jack_3.5mm, J2 mono_jack_3.5mm, J3 mono_jack_3.5mm, J4 mono_jack_3.5mm, J5 din5, J6 Conn_01x01, J7 rca, J8 2x20_Extra_Tall_Header, U1 MCP3008, U2 6N138

Commit message: update bom
Parts:
- J8: value 2x20_Extra_Tall_Header -> 2x20_Extra_Tall_Socket_Header
Changed lines of the file:
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@@
     (in_bom yes) (on_board yes)
     (property "Reference" "J8" (id 0) (at 264.16 140.335 0))
-    (property "Value" "2x20_Extra_Tall_Header" (id 1) (at 238.125 85.725 0))
+    (property "Value" "2x20_Extra_Tall_Socket_Header" (id 1) (at 238.125 85.725 0))
     (property "Footprint" "Connector_PinHeader_2.54mm:PinHeader_2x20_P2.54mm_Vertical" (id 2) (at 271.78 76.835 0)
       (effects (font (size 1.27 1.27)) hide)
@@
     )
     (path "/00000000-0000-0000-0000-00005c52f362"
-      (reference "J8") (unit 1) (value "2x20_Extra_Tall_Header") (footprint "Connector_PinHeader_2.54mm:PinHeader_2x20_P2.54mm_Vertical")
+      (reference "J8") (unit 1) (value "2x20_Extra_Tall_Socket_Header") (footprint "Connector_PinHeader_2.54mm:PinHeader_2x20_P2.54mm_Vertical")
     )
     (path "/00000000-0000-0000-0000-00005bc59626"
